File: sch/handy40choco/rpi_pico_mcu.kicad_sch (KiCad schematic)
At the start: 2 parts, among them Q1 DMG2301L, U1 Pico

Commit message: Kicad 9に変更しました。 マイコン基板から16ピンのピンヘッダに変更しました。
Connections:
- net DISPLAY_BL: no longer names the net of U1.26 (GPIO20)
- net DISPLAY_CS_N: no longer names the net of U1.22 (GPIO17)
- net DISPLAY_DATA: no longer names the net of U1.25 (GPIO19)
- net DISPLAY_DC: no longer names the net of U1.21 (GPIO16)
- net DISPLAY_RESET: no longer names the net of U1.29 (GPIO22)
- net DISPLAY_SCLK: no longer names the net of U1.24 (GPIO18)
- net DISPLAY_TE: no longer names the net of U1.27 (GPIO21)
- net LCD_RESET: no longer names the net of U1.30 (RUN)
- no-connect marks 7 -> 13
Changed lines of the file:
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@@
 (kicad_sch
-	(version 20231120)
+	(version 20250114)
 	(generator "eeschema")
-	(generator_version "8.0")
+	(generator_version "9.0")
 	(paper "A4")
 	(junction
@@
 	)
 	(no_connect
-		(at 124.46 76.2)
-	)
-	(no_connect
-		(at 124.46 78.74)
+		(at 160.02 104.14)
+	)
+	(no_connect
+		(at 160.02 111.76)
 	)
 	(no_connect
@@
 	)
 	(no_connect
+		(at 160.02 114.3)
+	)
+	(no_connect
+		(at 160.02 124.46)
+	)
+	(no_connect
+		(at 160.02 116.84)
+	)
+	(no_connect
+		(at 160.02 101.6)
+	)
+	(no_connect
+		(at 160.02 121.92)
+	)
+	(no_connect
+		(at 160.02 109.22)
+	)
+	(no_connect
 		(at 160.02 83.82)
 	)
@@
 	(wire
 		(pts
-			(xy 160.02 109.22) (xy 195.58 109.22)
-		)
-		(stroke
-			(width 0)
-			(type default)
-		)
-	)
-	(wire
-		(pts
-			(xy 160.02 101.6) (xy 195.58 101.6)
-		)
-		(stroke
-			(width 0)
-			(type default)
-		)
-	)
-	(wire
-		(pts
 			(xy 100.33 124.46) (xy 124.46 124.46)
 		)
@@
 	(wire
 		(pts
-			(xy 160.02 121.92) (xy 195.58 121.92)
-		)
-		(stroke
-			(width 0)
-			(type default)
-		)
-	)
-	(wire
-		(pts
 			(xy 142.24 58.42) (xy 142.24 55.88)
 		)
@@
 	(wire
 		(pts
-			(xy 160.02 124.46) (xy 195.58 124.46)
-		)
-		(stroke
-			(width 0)
-			(type default)
-		)
-	)
-	(wire
-		(pts
 			(xy 121.92 93.98) (xy 121.92 106.68)
 		)
@@
 	(wire
 		(pts
-			(xy 160.02 114.3) (xy 195.58 114.3)
-		)
-		(stroke
-			(width 0)
-			(type default)
-		)
-	)
-	(wire
-		(pts
 			(xy 100.33 99.06) (xy 124.46 99.06)
 		)
@@
 	(wire
 		(pts
-			(xy 160.02 104.14) (xy 195.58 104.14)
-		)
-		(stroke
-			(width 0)
-			(type default)
-		)
-	)
-	(wire
-		(pts
 			(xy 160.02 76.2) (xy 162.56 76.2)
 		)
@@
 	(wire
 		(pts
-			(xy 160.02 116.84) (xy 195.58 116.84)
-		)
-		(stroke
-			(width 0)
-			(type default)
-		)
-	)
-	(wire
-		(pts
 			(xy 162.56 106.68) (xy 162.56 119.38)
 		)
@@
 	(wire
 		(pts
-			(xy 160.02 111.76) (xy 195.58 111.76)
-		)
-		(stroke
-			(width 0)
-			(type default)
-		)
-	)
-	(wire
-		(pts
 			(xy 100.33 116.84) (xy 124.46 116.84)
 		)
@@
 		(shape bidirectional)
 		(at 100.33 116.84 180)
-		(fields_autoplaced yes)
-		(effects
-			(font
-				(size 1.27 1.27)
-			)
-			(justify right)
-		)
-	)
-	(hierarchical_label "DISPLAY_CS_N"
-		(shape output)
-		(at 195.58 121.92 0)
-		(fields_autoplaced yes)
-		(effects
-			(font
-				(size 1.27 1.27)
-			)
-			(justify left)
-		)
-	)
-	(hierarchical_label "DISPLAY_DATA"
-		(shape output)
-		(at 195.58 114.3 0)
-		(fields_autoplaced yes)
-		(effects
-			(font
-				(size 1.27 1.27)
-			)
-			(justify left)
+		(effects
+			(font
+				(size 1.27 1.27)
+			)
+			(justify right)
 		)
 	)
@@
 		(shape bidirectional)
 		(at 100.33 104.14 180)
-		(fields_autoplaced yes)
 		(effects
 			(font
@@
 		(shape bidirectional)
 		(at 100.33 99.06 180)
-		(fields_autoplaced yes)
 		(effects
 			(font
@@
 		(shape bidirectional)
 		(at 100.33 86.36 180)
-		(fields_autoplaced yes)
-		(effects
-			(font
-				(size 1.27 1.27)
-			)
-			(justify right)
-		)
-	)
-	(hierarchical_label "DISPLAY_SCLK"
-		(shape output)
-		(at 195.58 116.84 0)
-		(fields_autoplaced yes)
-		(effects
-			(font
-				(size 1.27 1.27)
-			)
-			(justify left)
+		(effects
+			(font
+				(size 1.27 1.27)
+			)
+			(justify right)
 		)
 	)
@@
 		(shape bidirectional)
 		(at 100.33 109.22 180)
-		(fields_autoplaced yes)
-		(effects
-			(font
-				(size 1.27 1.27)
-			)
-			(justify right)
-		)
-	)
-	(hierarchical_label "DISPLAY_DC"
-		(shape output)
-		(at 195.58 124.46 0)
-		(fields_autoplaced yes)
-		(effects
-			(font
-				(size 1.27 1.27)
-			)
-			(justify left)
+		(effects
+			(font
+				(size 1.27 1.27)
+			)
+			(justify right)
 		)
 	)
@@
 		(shape bidirectional)
 		(at 100.33 114.3 180)
-		(fields_autoplaced yes)
 		(effects
 			(font
@@
 		(shape bidirectional)
 		(at 100.33 124.46 180)
-		(fields_autoplaced yes)
 		(effects
 			(font
@@
 		(shape bidirectional)
 		(at 100.33 96.52 180)
-		(fields_autoplaced yes)
 		(effects
 			(font
@@
 		(shape bidirectional)
 		(at 100.33 101.6 180)
-		(fields_autoplaced yes)
 		(effects
 			(font
@@
 		(shape bidirectional)
 		(at 100.33 121.92 180)
-		(fields_autoplaced yes)
 		(effects
 			(font
@@
 		(shape input)
 		(at 116.84 48.26 180)
-		(fields_autoplaced yes)
-		(effects
-			(font
-				(size 1.27 1.27)
-			)
-			(justify right)
-		)
-	)
-	(hierarchical_label "DISPLAY_TE"
-		(shape output)
-		(at 195.58 109.22 0)
-		(fields_autoplaced yes)
-		(effects
-			(font
-				(size 1.27 1.27)
-			)
-			(justify left)
+		(effects
+			(font
+				(size 1.27 1.27)
+			)
+			(justify right)
 		)
 	)
@@
 		(shape bidirectional)
 		(at 100.33 83.82 180)
-		(fields_autoplaced yes)
 		(effects
 			(font
@@
 		(shape bidirectional)
 		(at 100.33 88.9 180)
-		(fields_autoplaced yes)
-		(effects
-			(font
-				(size 1.27 1.27)
-			)
-			(justify right)
-		)
-	)
-	(hierarchical_label "DISPLAY_BL"
-		(shape output)
-		(at 195.58 111.76 0)
-		(fields_autoplaced yes)
-		(effects
-			(font
-				(size 1.27 1.27)
-			)
-			(justify left)
+		(effects
+			(font
+				(size 1.27 1.27)
+			)
+			(justify right)
 		)
 	)
@@
 		(shape bidirectional)
 		(at 100.33 91.44 180)
-		(fields_autoplaced yes)
 		(effects
 			(font
@@
 		(shape bidirectional)
 		(at 100.33 111.76 180)
-		(fields_autoplaced yes)
-		(effects
-			(font
-				(size 1.27 1.27)
-			)
-			(justify right)
-		)
-	)
-	(hierarchical_label "DISPLAY_RESET"
-		(shape output)
-		(at 195.58 104.14 0)
-		(fields_autoplaced yes)
-		(effects
-			(font
-				(size 1.27 1.27)
-			)
-			(justify left)
-		)
-	)
-	(hierarchical_label "LCD_RESET"
-		(shape output)
-		(at 195.58 101.6 0)
-		(fields_autoplaced yes)
-		(effects
-			(font
-				(size 1.27 1.27)
-			)
-			(justify left)
-		)
-	)
+		(effects
+			(font
+				(size 1.27 1.27)
+			)
+			(justify right)
+		)
+	)
