File: sch/handy40choco/sw_matrix.kicad_sch (KiCad schematic)
At the start: 80 parts, among them SW1 SW_Push, SW10 SW_Push, SW11 SW_Push, SW12 SW_Push, SW13 SW_Push, SW14 SW_Push, SW15 SW_Push, SW16 SW_Push, SW17 SW_Push, SW18 SW_Push, SW19 SW_Push, SW2 SW_Push, SW20 SW_Push, SW21 SW_Push, SW22 SW_Push, SW23 SW_Push, SW24 SW_Push, SW25 SW_Push, SW26 SW_Push, SW27 SW_Push, SW28 SW_Push, SW29 SW_Push, SW3 SW_Push, SW30 SW_Push, SW31 SW_Push, SW32 SW_Push, SW33 SW_Push, SW34 SW_Push, SW35 SW_Push, SW36 SW_Push, SW37 SW_Push, SW38 SW_Push, SW39 SW_Push, SW4 SW_Push, SW40 SW_Push, SW5 SW_Push, SW6 SW_Push, SW7 SW_Push, SW8 SW_Push, SW9 SW_Push

Commit message: 配線を完了しました。 シルクの位置を調整しました。
Parts:
- SW1, SW10, SW11, SW12, SW13, SW14, SW15, SW16, SW17, SW18, SW19, SW2, SW20, SW21, SW22, SW23, SW24, SW25, SW26, SW27, SW28, SW29, SW3, SW30, SW31, SW32, SW33, SW34, SW35, SW36, SW37, SW38, SW39, SW4, SW40, SW5, SW6, SW7, SW8, SW9: footprint my_keyswitch:SW_Hotswap_Kailh_Choc_V1V2 -> my_keyswitch:SW_Hotswap_Kailh_Choc_V1V2_no_mp
Changed lines of the file:
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@@
 			)
 		)
-		(property "Footprint" "my_keyswitch:SW_Hotswap_Kailh_Choc_V1V2"
+		(property "Footprint" "my_keyswitch:SW_Hotswap_Kailh_Choc_V1V2_no_mp"
 			(at 34.29 96.52 0)
 			(effects
@@
 			)
 		)
-		(property "Footprint" "my_keyswitch:SW_Hotswap_Kailh_Choc_V1V2"
+		(property "Footprint" "my_keyswitch:SW_Hotswap_Kailh_Choc_V1V2_no_mp"
 			(at 95.25 50.8 0)
 			(effects
@@
 			)
 		)
-		(property "Footprint" "my_keyswitch:SW_Hotswap_Kailh_Choc_V1V2"
+		(property "Footprint" "my_keyswitch:SW_Hotswap_Kailh_Choc_V1V2_no_mp"
 			(at 176.53 119.38 0)
 			(effects
@@
 			)
 		)
-		(property "Footprint" "my_keyswitch:SW_Hotswap_Kailh_Choc_V1V2"
+		(property "Footprint" "my_keyswitch:SW_Hotswap_Kailh_Choc_V1V2_no_mp"
 			(at 54.61 119.38 0)
 			(effects
@@
 			)
 		)
-		(property "Footprint" "my_keyswitch:SW_Hotswap_Kailh_Choc_V1V2"
+		(property "Footprint" "my_keyswitch:SW_Hotswap_Kailh_Choc_V1V2_no_mp"
 			(at 176.53 96.52 0)
 			(effects
@@
 			)
 		)
-		(property "Footprint" "my_keyswitch:SW_Hotswap_Kailh_Choc_V1V2"
+		(property "Footprint" "my_keyswitch:SW_Hotswap_Kailh_Choc_V1V2_no_mp"
 			(at 156.21 96.52 0)
 			(effects
@@
 			)
 		)
-		(property "Footprint" "my_keyswitch:SW_Hotswap_Kailh_Choc_V1V2"
+		(property "Footprint" "my_keyswitch:SW_Hotswap_Kailh_Choc_V1V2_no_mp"
 			(at 176.53 73.66 0)
 			(effects
@@
 			)
 		)
-		(property "Footprint" "my_keyswitch:SW_Hotswap_Kailh_Choc_V1V2"
+		(property "Footprint" "my_keyswitch:SW_Hotswap_Kailh_Choc_V1V2_no_mp"
 			(at 74.93 50.8 0)
 			(effects
@@
 			)
 		)
-		(property "Footprint" "my_keyswitch:SW_Hotswap_Kailh_Choc_V1V2"
+		(property "Footprint" "my_keyswitch:SW_Hotswap_Kailh_Choc_V1V2_no_mp"
 			(at 156.21 119.38 0)
 			(effects
@@
 			)
 		)
-		(property "Footprint" "my_keyswitch:SW_Hotswap_Kailh_Choc_V1V2"
+		(property "Footprint" "my_keyswitch:SW_Hotswap_Kailh_Choc_V1V2_no_mp"
 			(at 74.93 119.38 0)
 			(effects
@@
 			)
 		)
-		(property "Footprint" "my_keyswitch:SW_Hotswap_Kailh_Choc_V1V2"
+		(property "Footprint" "my_keyswitch:SW_Hotswap_Kailh_Choc_V1V2_no_mp"
 			(at 34.29 119.38 0)
 			(effects
@@
 			)
 		)
-		(property "Footprint" "my_keyswitch:SW_Hotswap_Kailh_Choc_V1V2"
+		(property "Footprint" "my_keyswitch:SW_Hotswap_Kailh_Choc_V1V2_no_mp"
 			(at 54.61 96.52 0)
 			(effects
@@
 			)
 		)
-		(property "Footprint" "my_keyswitch:SW_Hotswap_Kailh_Choc_V1V2"
+		(property "Footprint" "my_keyswitch:SW_Hotswap_Kailh_Choc_V1V2_no_mp"
 			(at 95.25 119.38 0)
 			(effects
@@
 			)
 		)
-		(property "Footprint" "my_keyswitch:SW_Hotswap_Kailh_Choc_V1V2"
+		(property "Footprint" "my_keyswitch:SW_Hotswap_Kailh_Choc_V1V2_no_mp"
 			(at 156.21 50.8 0)
 			(effects
@@
 			)
 		)
-		(property "Footprint" "my_keyswitch:SW_Hotswap_Kailh_Choc_V1V2"
+		(property "Footprint" "my_keyswitch:SW_Hotswap_Kailh_Choc_V1V2_no_mp"
 			(at 54.61 50.8 0)
 			(effects
@@
 			)
 		)
-		(property "Footprint" "my_keyswitch:SW_Hotswap_Kailh_Choc_V1V2"
+		(property "Footprint" "my_keyswitch:SW_Hotswap_Kailh_Choc_V1V2_no_mp"
 			(at 74.93 73.66 0)
 			(effects
@@
 			)
 		)
-		(property "Footprint" "my_keyswitch:SW_Hotswap_Kailh_Choc_V1V2"
+		(property "Footprint" "my_keyswitch:SW_Hotswap_Kailh_Choc_V1V2_no_mp"
 			(at 115.57 50.8 0)
 			(effects
@@
 			)
 		)
-		(property "Footprint" "my_keyswitch:SW_Hotswap_Kailh_Choc_V1V2"
+		(property "Footprint" "my_keyswitch:SW_Hotswap_Kailh_Choc_V1V2_no_mp"
 			(at 156.21 73.66 0)
 			(effects
@@
 			)
 		)
-		(property "Footprint" "my_keyswitch:SW_Hotswap_Kailh_Choc_V1V2"
+		(property "Footprint" "my_keyswitch:SW_Hotswap_Kailh_Choc_V1V2_no_mp"
 			(at 217.17 119.38 0)
 			(effects
@@
 			)
 		)
-		(property "Footprint" "my_keyswitch:SW_Hotswap_Kailh_Choc_V1V2"
+		(property "Footprint" "my_keyswitch:SW_Hotswap_Kailh_Choc_V1V2_no_mp"
 			(at 217.17 50.8 0)
 			(effects
@@
 			)
 		)
-		(property "Footprint" "my_keyswitch:SW_Hotswap_Kailh_Choc_V1V2"
+		(property "Footprint" "my_keyswitch:SW_Hotswap_Kailh_Choc_V1V2_no_mp"
 			(at 196.85 50.8 0)
 			(effects
@@
 			)
 		)
-		(property "Footprint" "my_keyswitch:SW_Hotswap_Kailh_Choc_V1V2"
+		(property "Footprint" "my_keyswitch:SW_Hotswap_Kailh_Choc_V1V2_no_mp"
 			(at 135.89 119.38 0)
 			(effects
@@
 			)
 		)
-		(property "Footprint" "my_keyswitch:SW_Hotswap_Kailh_Choc_V1V2"
+		(property "Footprint" "my_keyswitch:SW_Hotswap_Kailh_Choc_V1V2_no_mp"
 			(at 176.53 50.8 0)
 			(effects
@@
 			)
 		)
-		(property "Footprint" "my_keyswitch:SW_Hotswap_Kailh_Choc_V1V2"
+		(property "Footprint" "my_keyswitch:SW_Hotswap_Kailh_Choc_V1V2_no_mp"
 			(at 34.29 50.8 0)
 			(effects
@@
 			)
 		)
-		(property "Footprint" "my_keyswitch:SW_Hotswap_Kailh_Choc_V1V2"
+		(property "Footprint" "my_keyswitch:SW_Hotswap_Kailh_Choc_V1V2_no_mp"
 			(at 196.85 73.66 0)
 			(effects
@@
 			)
 		)
-		(property "Footprint" "my_keyswitch:SW_Hotswap_Kailh_Choc_V1V2"
+		(property "Footprint" "my_keyswitch:SW_Hotswap_Kailh_Choc_V1V2_no_mp"
 			(at 115.57 119.38 0)
 			(effects
@@
 			)
 		)
-		(property "Footprint" "my_keyswitch:SW_Hotswap_Kailh_Choc_V1V2"
+		(property "Footprint" "my_keyswitch:SW_Hotswap_Kailh_Choc_V1V2_no_mp"
 			(at 196.85 96.52 0)
 			(effects
@@
 			)
 		)
-		(property "Footprint" "my_keyswitch:SW_Hotswap_Kailh_Choc_V1V2"
+		(property "Footprint" "my_keyswitch:SW_Hotswap_Kailh_Choc_V1V2_no_mp"
 			(at 115.57 96.52 0)
 			(effects
@@
 			)
 		)
-		(property "Footprint" "my_keyswitch:SW_Hotswap_Kailh_Choc_V1V2"
+		(property "Footprint" "my_keyswitch:SW_Hotswap_Kailh_Choc_V1V2_no_mp"
 			(at 74.93 96.52 0)
 			(effects
@@
 			)
 		)
-		(property "Footprint" "my_keyswitch:SW_Hotswap_Kailh_Choc_V1V2"
+		(property "Footprint" "my_keyswitch:SW_Hotswap_Kailh_Choc_V1V2_no_mp"
 			(at 115.57 73.66 0)
 			(effects
@@
 			)
 		)
-		(property "Footprint" "my_keyswitch:SW_Hotswap_Kailh_Choc_V1V2"
+		(property "Footprint" "my_keyswitch:SW_Hotswap_Kailh_Choc_V1V2_no_mp"
 			(at 135.89 96.52 0)
 			(effects
@@
 			)
 		)
-		(property "Footprint" "my_keyswitch:SW_Hotswap_Kailh_Choc_V1V2"
+		(property "Footprint" "my_keyswitch:SW_Hotswap_Kailh_Choc_V1V2_no_mp"
 			(at 135.89 50.8 0)
 			(effects
@@
 			)
 		)
-		(property "Footprint" "my_keyswitch:SW_Hotswap_Kailh_Choc_V1V2"
+		(property "Footprint" "my_keyswitch:SW_Hotswap_Kailh_Choc_V1V2_no_mp"
 			(at 217.17 73.66 0)
 			(effects
@@
 			)
 		)
-		(property "Footprint" "my_keyswitch:SW_Hotswap_Kailh_Choc_V1V2"
+		(property "Footprint" "my_keyswitch:SW_Hotswap_Kailh_Choc_V1V2_no_mp"
 			(at 217.17 96.52 0)
 			(effects
@@
 			)
 		)
-		(property "Footprint" "my_keyswitch:SW_Hotswap_Kailh_Choc_V1V2"
+		(property "Footprint" "my_keyswitch:SW_Hotswap_Kailh_Choc_V1V2_no_mp"
 			(at 135.89 73.66 0)
 			(effects
@@
 			)
 		)
-		(property "Footprint" "my_keyswitch:SW_Hotswap_Kailh_Choc_V1V2"
+		(property "Footprint" "my_keyswitch:SW_Hotswap_Kailh_Choc_V1V2_no_mp"
 			(at 95.25 96.52 0)
 			(effects
@@
 			)
 		)
-		(property "Footprint" "my_keyswitch:SW_Hotswap_Kailh_Choc_V1V2"
+		(property "Footprint" "my_keyswitch:SW_Hotswap_Kailh_Choc_V1V2_no_mp"
 			(at 196.85 119.38 0)
 			(effects
@@
 			)
 		)
-		(property "Footprint" "my_keyswitch:SW_Hotswap_Kailh_Choc_V1V2"
+		(property "Footprint" "my_keyswitch:SW_Hotswap_Kailh_Choc_V1V2_no_mp"
 			(at 34.29 73.66 0)
 			(effects
@@
 			)
 		)
-		(property "Footprint" "my_keyswitch:SW_Hotswap_Kailh_Choc_V1V2"
+		(property "Footprint" "my_keyswitch:SW_Hotswap_Kailh_Choc_V1V2_no_mp"
 			(at 54.61 73.66 0)
 			(effects
@@
 			)
 		)
-		(property "Footprint" "my_keyswitch:SW_Hotswap_Kailh_Choc_V1V2"
+		(property "Footprint" "my_keyswitch:SW_Hotswap_Kailh_Choc_V1V2_no_mp"
 			(at 95.25 73.66 0)
 			(effects

Commit message: 左端のキーの向きを180度回転させて、基板幅を短くしました。
Connections:
- net COL0: now also SW1.1, SW11.1, SW21.1, SW31.1; no longer SW1.2, SW11.2, SW21.2, SW31.2
- net at D21.2 (A): now also SW21.2; no longer SW21.1
- net at D31.2 (A): now also SW31.2; no longer SW31.1
- net at D11.2 (A): now also SW11.2; no longer SW11.1
- net at D1.2 (A): now also SW1.2; no longer SW1.1
Changed lines of the file:
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@@
 		(lib_id "Switch:SW_Push")
 		(at 34.29 101.6 0)
+		(mirror y)
 		(unit 1)
 		(exclude_from_sim no)
@@
 		(on_board yes)
 		(dnp no)
-		(fields_autoplaced yes)
 		(property "Reference" "SW21"
 			(at 34.29 93.98 0)
@@
 		(lib_id "Switch:SW_Push")
 		(at 34.29 124.46 0)
+		(mirror y)
 		(unit 1)
 		(exclude_from_sim no)
@@
 		(on_board yes)
 		(dnp no)
-		(fields_autoplaced yes)
 		(property "Reference" "SW31"
 			(at 34.29 116.84 0)
@@
 		(lib_id "Switch:SW_Push")
 		(at 34.29 55.88 0)
+		(mirror y)
 		(unit 1)
 		(exclude_from_sim no)
@@
 		(on_board yes)
 		(dnp no)
-		(fields_autoplaced yes)
 		(property "Reference" "SW1"
 			(at 34.29 48.26 0)
@@
 		(lib_id "Switch:SW_Push")
 		(at 34.29 78.74 0)
+		(mirror y)
 		(unit 1)
 		(exclude_from_sim no)
@@
 		(on_board yes)
 		(dnp no)
-		(fields_autoplaced yes)
 		(property "Reference" "SW11"
 			(at 34.29 71.12 0)
