File: sch/handy40choco-mcu-esp32/handy40choco-mcu-esp32.kicad_pcb (KiCad board)
At the start: 2 copper layers, 175 x 112 mm, 147 parts, among them J1 Conn_01x02, J2 Conn_02x08_Odd_Even, J3 USB_C_Receptacle_USB2.0_16P, J4 Conn_01x04, Q1 DMG2301L, SW1 SW_Push, SW10 SW_Push, SW11 SW_Push, SW12 SW_Push, SW13 SW_Push, SW14 SW_Push, SW15 SW_Push, SW16 SW_Push, SW17 SW_Push, SW18 SW_Push, SW19 SW_Push, SW2 SW_Push, SW20 SW_Push, SW21 SW_Push, SW22 SW_Push, SW23 SW_Push, SW24 SW_Push, SW25 SW_Push, SW26 SW_Push, SW27 SW_Push, SW28 SW_Push, SW29 SW_Push, SW3 SW_Push, SW30 SW_Push, SW31 SW_Push, SW32 SW_Push, SW33 SW_Push, SW34 SW_Push, SW35 SW_Push, SW36 SW_Push, SW37 SW_Push, SW38 SW_Push, SW39 SW_Push, SW4 SW_Push, SW40 SW_Push, SW41 SW_Push, SW42 SW_Push, SW5 SW_Push, SW6 SW_Push, SW7 SW_Push, SW8 SW_Push, SW9 SW_Push, U1 Pico, U2 pimoroni lcd, U3 ESP32-S3-WROOM-1, U4 MIC5219-3.3YM5, Y1 32k

Commit message: マイコン基板(ESP32-S3)の雛形です。
Parts:
- removed D10, D11, D12, D13, D14, D15, D16, D17, D18, D19, D20, D21, D22, D23, D24, D25, D26, D27, D28, D29, D30, D31, D32, D33, D34, D35, D36, D37, D38, D39, D40, D7, D8, D9: 1N4148W, Diode_SMD:D_SOD-123
- removed D41, D42, D43: D_Schottky, Diode_SMD:D_SOD-123
- removed D44, D45, D46: D_TVS, Diode_SMD:D_SOD-123
- removed D47, D48, D49, D50, D51, D52, D53: LED, LED_SMD:LED_0603_1608Metric_Pad1.05x0.95mm_HandSolder
- removed H1, H10, H11, H12, H13, H14, H2, H3, H4, H5, H6, H7, H8, H9: MountingHole, my_keyswitch:my_MountingHole_2.2mm_M2
- removed Q1: DMG2301L, Package_TO_SOT_SMD:SOT-23
- removed R10: [10M], Resistor_SMD:R_0603_1608Metric
- removed R11, R12, R9: 0, Resistor_SMD:R_0603_1608Metric
- removed R13, R14, R15, R16, R17, R18, R19: 1k, Resistor_SMD:R_0603_1608Metric
- removed SW10, SW11, SW12, SW13, SW14, SW15, SW16, SW17, SW18, SW19, SW20, SW21, SW22, SW23, SW24, SW25, SW26, SW27, SW28, SW29, SW3, SW30, SW31, SW32, SW33, SW34, SW35, SW36, SW37, SW38, SW39, SW4, SW40, SW5, SW6, SW7, SW8, SW9: SW_Push, my_keyswitch:SW_Hotswap_Kailh_Choc_V1V2
- removed SW41, SW42: SW_Push, Button_Switch_SMD:SW_Push_SPST_NO_Alps_SKRK
- removed U3: ESP32-S3-WROOM-1, RF_Module:ESP32-S3-WROOM-1
- removed U4: MIC5219-3.3YM5, Package_TO_SOT_SMD:SOT-23-5
- C1: value 10u -> 10n
- C2: value 100n -> 15p
- C3: value 100n -> 470p
- C4: value 1u -> 15p
- C5: value 470p -> 100n
- C6: value 10n -> 1u
- C7: value 15p -> 10u
- C8: value 15p -> 100n
- D1, D2, D5: value 1N4148W -> D_Schottky; moved to F.Cu
- D3, D4, D6: value 1N4148W -> D_TVS; moved to F.Cu
- J2: value Conn_02x08_Odd_Even -> USB_C_Receptacle_USB2.0_16P; footprint my_pico:oled_PinSocket_2x08_P2.54mm_Vertical -> Connector_USB:USB_C_Receptacle_XKB_U262-16XN-4BVC11
- J3: value USB_C_Receptacle_USB2.0_16P -> Conn_01x04; footprint Connector_USB:USB_C_Receptacle_XKB_U262-16XN-4BVC11 -> Connector_JST:JST_XH_B4B-XH-A_1x04_P2.50mm_Vertical
- J4: value Conn_01x04 -> Conn_01x20; footprint Connector_JST:JST_XH_B4B-XH-A_1x04_P2.50mm_Vertical -> Connector_PinHeader_2.54mm:PinHeader_1x20_P2.54mm_Vertical
- R1, R2: value 0 -> 5.1k; moved to F.Cu
- R3: moved to F.Cu
- R4: value 10k -> [10M]; moved to F.Cu
- R5, R6: value 5.1k -> 0
- R7: value 10k -> 0
- SW1, SW2: footprint my_keyswitch:SW_Hotswap_Kailh_Choc_V1V2 -> Button_Switch_SMD:SW_Push_SPST_NO_Alps_SKRK
- U1: value Pico -> MIC5219-3.3YM5; footprint my_pico:pico_no_dbg_smd_th_p0.85 -> Package_TO_SOT_SMD:SOT-23-5
- U2: value pimoroni lcd -> ESP32-S3-WROOM-1; footprint my_pico:pimoroni_lcd_p0.85 -> RF_Module:ESP32-S3-WROOM-1
- moved J4 286.3 mm to (235.0, 87.5), turned to -90 degrees
- moved R5 219.8 mm to (157.0, 69.5)
- moved R6 219.8 mm to (157.0, 72.0)
- moved R7 219.8 mm to (157.0, 74.5)
- moved R8 219.8 mm to (157.0, 77.0)
- moved C1 183.6 mm to (161.1, 59.4)
- moved C2 183.6 mm to (161.1, 61.9)
- moved C3 183.6 mm to (161.1, 64.5)
- moved C4 183.6 mm to (161.1, 67.0)
- moved C5 183.6 mm to (161.1, 69.5)
- moved C6 183.6 mm to (161.1, 72.0)
- moved C7 183.6 mm to (161.1, 74.5)
- moved C8 183.6 mm to (161.1, 77.0)
- moved Y1 169.7 mm to (148.1, 84.5)
- moved F1 129.4 mm to (110.0, 68.0)
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Connections:
- C1 pad 1: +3.3VP -> /EN
- C2 pad 1: +3.3VP -> Net-(C2-Pad1)
- C3 pad 1: +3.3VP -> Net-(U1-BP)
- C4 pad 1: +3.3VP -> Net-(C4-Pad1)
- C5 pad 1: Net-(U4-BP) -> +3.3VP
- C6 pad 1: /ESP32-S3 mcu/EN -> +3.3VP
- C7 pad 1: Net-(C7-Pad1) -> +3.3VP
- C8 pad 1: Net-(C8-Pad1) -> +3.3VP
- D1 pad 1: /ROW0 -> Net-(D1-K)
- D1 pad 2: Net-(D1-A) -> /VBUS
- D2 pad 1: /ROW0 -> Net-(D1-K)
- D2 pad 2: Net-(D2-A) -> /VBAT
- D3 pad 1: /ROW0 -> GND
- D3 pad 2: Net-(D3-A) -> Net-(D3-A2)
- D4 pad 1: /ROW0 -> GND
- D4 pad 2: Net-(D4-A) -> /USB_P
- D5 pad 1: /ROW0 -> Net-(D1-K)
- D5 pad 2: Net-(D5-A) -> +3.3VP
- D6 pad 1: /ROW0 -> GND
- D6 pad 2: Net-(D6-A) -> /USB_M
- F1 pad 1: Net-(D46-A2) -> Net-(D3-A2)
- F1 pad 2: /ESP32-S3 mcu/VBUS -> /VBUS
- J4 pad 1: +3.3VP -> /ROW3
- J4 pad 2: Net-(J4-Pin_2) -> /ROW2
- J4 pad 3: Net-(J4-Pin_3) -> GND
- J4 pad 4: GND -> /ROW1
- R1 pad 1: Net-(J2-Pin_13) -> Net-(J2-CC2)
- R2 pad 1: Net-(J2-Pin_12) -> Net-(J2-CC1)
- R3 pad 1: +3.3V -> +3.3VP
- R3 pad 2: /OLED_RESET -> /EN
- R4 pad 1: +3.3V -> Net-(C2-Pad1)
- R4 pad 2: /CS_N -> Net-(C4-Pad1)
- R5 pad 1: Net-(J3-CC2) -> Net-(C2-Pad1)
- R5 pad 2: GND -> /XTAL_P
- R6 pad 1: Net-(J3-CC1) -> Net-(C4-Pad1)
- R6 pad 2: GND -> /XTAL_N
- R7 pad 1: +3.3VP -> /TXD0
- R7 pad 2: /ESP32-S3 mcu/EN -> Net-(J3-Pin_2)
- R8 pad 1: Net-(U3-TXD0) -> /RXD0
- R8 pad 2: Net-(J4-Pin_2) -> Net-(J3-Pin_3)
- SW1 pad 1: Net-(D1-A) -> GND
- SW1 pad 2: /COL0 -> /EN
- SW2 pad 1: Net-(D2-A) -> GND
- SW2 pad 2: /COL1 -> /IO0
- U1 pad 1: unconnected-(U1-GPIO0-Pad1)_1 -> Net-(D1-K)
- U1 pad 2: unconnected-(U1-GPIO1-Pad2)_1 -> GND
- U1 pad 3: GND -> Net-(D1-K)
- U1 pad 4: /ROW3 -> Net-(U1-BP)
- U1 pad 5: /ROW2 -> +3.3VP
- U2 pad 1: unconnected-(U2-NC0-Pad1) -> GND
- U2 pad 10: unconnected-(U2-PWRKEY_BL-Pad10) -> /COL4
- U2 pad 11: unconnected-(U2-UART_TX_DC-Pad11) -> /COL5
- U2 pad 12: unconnected-(U2-UART_RX_CS-Pad12) -> /COL6
- U2 pad 13: GND -> /USB_M
- U2 pad 14: unconnected-(U2-NETLIGHT_SCK-Pad14) -> /USB_P
- U2 pad 17: unconnected-(U2-SWB-Pad17) -> /COL7
- U2 pad 18: GND -> /COL8
- U2 pad 19: unconnected-(U2-SWX-Pad19) -> /COL9
- U2 pad 2: unconnected-(U2-NC1-Pad2) -> +3.3VP
- U2 pad 20: unconnected-(U2-SWY-Pad20) -> /COL10
- U2 pad 21: /DC -> /COL11
- U2 pad 22: /CS_N -> /ROW0
- U2 pad 23: GND -> /ROW1
- U2 pad 24: /SCLK -> /ROW3
- U2 pad 25: /DATA -> /ROW2
- U2 pad 26: /LCD_BL -> unconnected-(U2-IO45-Pad26)
- U2 pad 27: /LCD_TE -> /IO0
- U2 pad 28: GND -> unconnected-(U2-IO35-Pad28)
- U2 pad 3: GND -> /EN
- U2 pad 30: /LCD_RESET -> unconnected-(U2-IO37-Pad30)
- U2 pad 33: GND -> unconnected-(U2-IO40-Pad33)
- U2 pad 36: +3.3V -> /RXD0
- U2 pad 37: unconnected-(U2-NC6-Pad37) -> /TXD0
- U2 pad 38: GND -> unconnected-(U2-IO2-Pad38)
- U2 pad 4: unconnected-(U2-NC2-Pad4) -> /COL0
- U2 pad 40: unconnected-(U2-NC7-Pad40) -> GND
- U2 pad 5: unconnected-(U2-NC3-Pad5) -> /COL1
- U2 pad 6: unconnected-(U2-I2C_SDA-Pad6) -> /COL2
- U2 pad 7: unconnected-(U2-I2C_SCL-Pad7) -> /COL3
- U2 pad 8: GND -> /XTAL_P
- U2 pad 9: unconnected-(U2-NC4-Pad9) -> /XTAL_N
- Y1 pad 1: Net-(C7-Pad1) -> Net-(C2-Pad1)
- Y1 pad 2: Net-(C8-Pad1) -> Net-(C4-Pad1)
Routing:
- net /ROW3: track 291.0 -> 0.00 mm, vias 10 -> 0
- net /ROW2: track 274.4 -> 0.00 mm, vias 10 -> 0
- net /ROW1: track 259.9 -> 0.00 mm, vias 10 -> 0
- net /ROW0: track 224.4 -> 0.00 mm, vias 10 -> 0
- net /COL0: track 216.7 -> 0.00 mm
- net /COL1: track 206.4 -> 0.00 mm
- net /COL2: track 186.6 -> 0.00 mm
- net /COL3: track 173.0 -> 0.00 mm
- net +3.3V: track 170.8 -> 0.00 mm, vias 3 -> 0
- net /COL4: track 155.4 -> 0.00 mm
- net /COL5: track 142.1 -> 0.00 mm
- net /COL6: track 132.1 -> 0.00 mm
- net /COL7: track 119.2 -> 0.00 mm
- net /LCD_RESET: track 111.5 -> 0.00 mm
- net /COL8: track 107.2 -> 0.00 mm
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Other:
- board size 175 x 112 mm -> 169.5 x 40 mm
- board text added: "handy40choco mcu esp32 rev.1"
- board text added: "https://github.com/kenyahiro/handy40choco"
- board text removed: "https://github.com/kenyahiro/mini48-keyboard"
- board text removed: "mini48-keyboard_v2_p17"
